File: PCB/PCB_ControlLamparasSonido.kicad_pcb (KiCad board)
At the start: 2 copper layers, 87 x 39 mm, 38 parts, among them P1 Power, P2 Carga, Q1 BC549, Q2 BC549, Q3 BC557, Q4 BC547, Q5 BC547, Q6 BT136-500

Commit message: Finalizado
Proyecto Finalizado
Parts:
- moved P1 5.39 mm to (79.0, 51.0)
- moved P2 2.00 mm to (156.0, 58.0)
Routing:
- net Net-(Q6-A2): track 35.2 -> 37.2 mm
Changed lines of the file:
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@@
 	(footprint "BORNERA_2:TE_282837-2"
 		(layer "F.Cu")
-		(at 154 58 90)
+		(at 156 58 90)
 		(property "Reference" "P2"
 			(at -1.127255 -5.614945 90)
@@
 	(footprint "BORNERA_2:TE_282837-2"
 		(layer "F.Cu")
-		(at 84 49 -90)
+		(at 79 51 -90)
 		(property "Reference" "P1"
 			(at -5 -6 90)
@@
 		)
 	)
-	(gr_circle
-		(center 154 71)
-		(end 157 71)
-		(stroke
-			(width 0.1)
-			(type solid)
-		)
-		(fill yes)
-		(layer "F.SilkS")
-	)
-	(gr_circle
-		(center 81 60)
-		(end 84 60)
-		(stroke
-			(width 0.1)
-			(type solid)
-		)
-		(fill yes)
-		(layer "F.SilkS")
-	)
-	(gr_circle
-		(center 154 46)
-		(end 157 46)
-		(stroke
-			(width 0.1)
-			(type solid)
-		)
-		(fill yes)
-		(layer "F.SilkS")
-	)
 	(gr_line
 		(start 154 78)
@@
 	)
 	(gr_text "+"
-		(at 159 56 0)
-		(layer "F.SilkS")
+		(at 155 52 0)
+		(layer "F.SilkS" knockout)
 		(effects
 			(font
@@
 	(gr_text "230V AC"
 		(at 82 42 0)
-		(layer "F.SilkS")
+		(layer "F.SilkS" knockout)
 		(effects
 			(font
@@
 	)
 	(gr_text "Controlador de Lampara por Sonido"
-		(at 103 76 0)
+		(at 97 76 0)
 		(layer "F.SilkS" knockout)
 		(effects
@@
 	)
 	(gr_text "+"
-		(at 77 47 0)
-		(layer "F.SilkS")
+		(at 79 45 0)
+		(layer "F.SilkS" knockout)
 		(effects
 			(font
@@
 	)
 	(segment
-		(start 154 60.54)
-		(end 140.46 60.54)
+		(start 121.055 66)
+		(end 135 66)
 		(width 0.9)
 		(layer "F.Cu")
@@
 	)
 	(segment
-		(start 140.46 60.54)
-		(end 135 66)
+		(start 135 66)
+		(end 140.46 60.54)
 		(width 0.9)
 		(layer "F.Cu")
@@
 	)
 	(segment
-		(start 135 66)
-		(end 121.055 66)
+		(start 140.46 60.54)
+		(end 156 60.54)
 		(width 0.9)
 		(layer "F.Cu")
