File: PCB/PCB_ControlLamparasSonido.kicad_sch (KiCad schematic)
At the start: 34 parts, among them P1 Power, P2 Carga, Q1 BC549, Q2 BC549, Q3 BC557, Q4 BC547, Q5 BC547, Q6 BT136-500

Commit message: PCB
Diseño terminado de la PCB 2 capas
Parts:
- added H1, H2, H3: MountingHole_Pad, MountingHole:MountingHole_2.2mm_M2_ISO7380_Pad, symbol Mechanical:MountingHole_Pad
Connections:
- net GND: now also H1.1, H2.1, H3.1
Other:
- note added: "Pads de montaje"
